File: schematics/globals.kicad_sch (KiCad schematic)
At the start: 35 parts, among them J1 Power, U1 74HCU04, U2 74HC14, U3 ATF22V10C-7, U4 74HC590, U5 74HC590, U6 74HC590, U7 PicoROM32, Y1 12MHz

Commit message: updating schematics as I wire the board
Connections:
- net GND: now also U2.11, U2.9, U7.1 (A18), U7.30 (A17); no longer U2.3, U2.5
- net at D3.2 (A), R6.1, U3.4 (~{R_IN})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: now also U2.5; no longer U2.11
- net at C7.1, D2.2 (A), R5.2: now also U2.3; no longer U2.9
- net at D3.1 (K): now also U2.4; no longer U2.8
- net at D4.1 (K): now also U2.6; no longer U2.10
Changed lines of the file:
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@@
 	)
 	(junction
+		(at 214.63 91.44)
+		(diameter 0)
+		(color 0 0 0 0)
+	)
+	(junction
 		(at 208.28 58.42)
 		(diameter 0)
@@
 	)
 	(junction
+		(at 214.63 93.98)
+		(diameter 0)
+		(color 0 0 0 0)
+	)
+	(junction
 		(at 40.64 27.94)
 		(diameter 0)
@@
 	(wire
 		(pts
+			(xy 214.63 91.44) (xy 217.17 91.44)
+		)
+		(stroke
+			(width 0)
+			(type default)
+		)
+	)
+	(wire
+		(pts
 			(xy 180.34 25.4) (xy 180.34 45.72)
 		)
@@
 	(wire
 		(pts
-			(xy 214.63 88.9) (xy 214.63 109.22)
+			(xy 214.63 88.9) (xy 214.63 91.44)
 		)
 		(stroke
@@
 	(wire
 		(pts
+			(xy 214.63 91.44) (xy 214.63 93.98)
+		)
+		(stroke
+			(width 0)
+			(type default)
+		)
+	)
+	(wire
+		(pts
 			(xy 72.39 33.02) (xy 72.39 27.94)
 		)
@@
 	(wire
 		(pts
+			(xy 214.63 93.98) (xy 217.17 93.98)
+		)
+		(stroke
+			(width 0)
+			(type default)
+		)
+	)
+	(wire
+		(pts
 			(xy 43.18 95.25) (xy 49.53 95.25)
 		)
@@
 	(wire
 		(pts
+			(xy 214.63 93.98) (xy 214.63 109.22)
+		)
+		(stroke
+			(width 0)
+			(type default)
+		)
+	)
+	(wire
+		(pts
 			(xy 194.31 149.86) (xy 194.31 86.36)
 		)
@@
 		(lib_id "74xx:74HC14")
 		(at 64.77 190.5 90)
-		(unit 2)
+		(unit 4)
 		(body_style 1)
 		(exclude_from_sim no)
@@
 				(path "/94c72abe-aaa5-49aa-8ab7-5d3e7cbc10be/560ef1bd-4b3f-459c-9f6a-9898850b3c5b"
 					(reference "U2")
-					(unit 2)
+					(unit 4)
 				)
 			)
@@
 		(lib_id "74xx:74HC14")
 		(at 97.79 72.39 0)
-		(unit 5)
+		(unit 3)
 		(body_style 1)
 		(exclude_from_sim no)
@@
 		(dnp no)
 		(property "Reference" "U2"
-			(at 97.79 68.58 0)
+			(at 97.79 66.04 0)
 			(show_name no)
 			(do_not_autoplace no)
@@
 		)
 		(property "Value" "74HC14"
-			(at 97.79 66.04 0)
+			(at 97.79 68.58 0)
 			(show_name no)
 			(do_not_autoplace no)
@@
 				(path "/94c72abe-aaa5-49aa-8ab7-5d3e7cbc10be/560ef1bd-4b3f-459c-9f6a-9898850b3c5b"
 					(reference "U2")
-					(unit 5)
+					(unit 3)
 				)
 			)
@@
 		(lib_id "74xx:74HC14")
 		(at 76.2 190.5 90)
-		(unit 3)
+		(unit 5)
 		(body_style 1)
 		(exclude_from_sim no)
@@
 				(path "/94c72abe-aaa5-49aa-8ab7-5d3e7cbc10be/560ef1bd-4b3f-459c-9f6a-9898850b3c5b"
 					(reference "U2")
-					(unit 3)
+					(unit 5)
 				)
 			)
@@
 		(lib_id "74xx:74HC14")
 		(at 74.93 64.77 0)
-		(unit 4)
+		(unit 2)
 		(body_style 1)
 		(exclude_from_sim no)
@@
 				(path "/94c72abe-aaa5-49aa-8ab7-5d3e7cbc10be/560ef1bd-4b3f-459c-9f6a-9898850b3c5b"
 					(reference "U2")
-					(unit 4)
+					(unit 2)
 				)
 			)
