File: schematics/cpu.kicad_sch (KiCad schematic)
At the start: 12 parts, among them U8 W65C02SxP

Commit message: clock improvements
Connections:
- net ϕ2 renamed ϕ2.1
Changed lines of the file:
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@@
 		)
 	)
-	(global_label "ϕ2"
+	(global_label "ϕ2.1"
 		(shape input)
 		(at 107.95 73.66 180)
@@
 		)
 		(property "Intersheetrefs" "${INTERSHEET_REFS}"
-			(at 102.4248 73.66 0)
+			(at 100.6105 73.66 0)
 			(hide yes)
 			(show_name no)
