File: schematics/uart.kicad_sch (KiCad schematic)
At the start: 4 parts, among them U15 W65C51NxP, Y2 1.8432MHz

Commit message: clock improvements
Connections:
- net ϕ2 renamed ϕ2.0
Changed lines of the file:
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@@
 		)
 	)
-	(global_label "ϕ2"
+	(global_label "ϕ2.0"
 		(shape input)
 		(at 121.92 81.28 180)
@@
 		)
 		(property "Intersheetrefs" "${INTERSHEET_REFS}"
-			(at 116.3948 81.28 0)
+			(at 114.5805 81.28 0)
 			(hide yes)
 			(show_name no)
