File: schematics/via.kicad_sch (KiCad schematic)
At the start: 31 parts, among them SW2 SW_DIP_x08, SW7 SW_DIP_x08, U16 74HC14, U17 W65C22SxP

Commit message: clock improvements
Connections:
- net ϕ2 renamed ϕ2.0
Other:
- moved on the sheet: D16
Changed lines of the file:
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@@
 	(wire
 		(pts
-			(xy 101.6 85.09) (xy 109.22 85.09)
+			(xy 99.06 85.09) (xy 109.22 85.09)
 		)
 		(stroke
@@
 	(wire
 		(pts
-			(xy 92.71 85.09) (xy 93.98 85.09)
+			(xy 90.17 85.09) (xy 91.44 85.09)
 		)
 		(stroke
@@
 		)
 	)
-	(global_label "ϕ2"
+	(global_label "ϕ2.0"
 		(shape input)
 		(at 106.68 81.28 180)
@@
 		)
 		(property "Intersheetrefs" "${INTERSHEET_REFS}"
-			(at 101.1548 81.28 0)
+			(at 99.3405 81.28 0)
 			(hide yes)
 			(show_name no)
@@
 	(global_label "~{IRQ}"
 		(shape output)
-		(at 92.71 85.09 180)
+		(at 90.17 85.09 180)
 		(fields_autoplaced yes)
 		(effects
@@
 		)
 		(property "Intersheetrefs" "${INTERSHEET_REFS}"
-			(at 86.5195 85.09 0)
+			(at 83.9795 85.09 0)
 			(hide yes)
 			(show_name no)
@@
 	(symbol
 		(lib_id "Diode:1N4148")
-		(at 97.79 85.09 180)
+		(at 95.25 85.09 180)
 		(unit 1)
 		(body_style 1)
@@
 		(dnp no)
 		(property "Reference" "D16"
-			(at 97.79 80.01 0)
+			(at 95.25 80.01 0)
 			(show_name no)
 			(do_not_autoplace no)
@@
 		)
 		(property "Value" "1N4148"
-			(at 97.79 82.55 0)
+			(at 95.25 82.55 0)
 			(show_name no)
 			(do_not_autoplace no)
@@
 		)
 		(property "Footprint" "Diode_THT:D_DO-35_SOD27_P7.62mm_Horizontal"
-			(at 97.79 85.09 0)
+			(at 95.25 85.09 0)
 			(hide yes)
 			(show_name no)
@@
 		)
 		(property "Datasheet" "https://assets.nexperia.com/documents/data-sheet/1N4148_1N4448.pdf"
-			(at 97.79 85.09 0)
+			(at 95.25 85.09 0)
 			(hide yes)
 			(show_name no)
@@
 		)
 		(property "Description" "100V 0.15A standard switching diode, DO-35"
-			(at 97.79 85.09 0)
+			(at 95.25 85.09 0)
 			(hide yes)
 			(show_name no)
@@
 		)
 		(property "Sim.Device" "D"
-			(at 97.79 85.09 0)
+			(at 95.25 85.09 0)
 			(hide yes)
 			(show_name no)
@@
 		)
 		(property "Sim.Pins" "1=K 2=A"
-			(at 97.79 85.09 0)
-			(hide yes)
-			(show_name no)
+			(at 95.25 85.09 0)
+			(hide yes)
+			(show_name no)
